Commit message: AI update

File: URDF/URDF.urdf (robot description, URDF)
Before this commit: robot URDF, 7 links, 6 joints
Joints:
- joint Revolute_1: axis -0.126869 -0.002806 0.991916 -> 0.126869 0.002806 -0.991916
- joint Revolute_2: axis -0.022114 0.999755 -0.0 -> 0.022114 -0.999755 0.0
- joint Revolute_3: axis -0.0 -0.0 -1.0 -> 0.0 0.0 1.0; origin xyz=-0.562444 0.0 -0.0175 rpy=0 0 0 -> xyz=0.562444 0.0 -0.0175 rpy=0 0 0
